Commit message: Fix some init bug.

File: bipedal_wheel_description/urdf/leg.urdf.xacro (robot description, xacro)
@@ -24,5 +24,4 @@
             <parent link="${connected_to}"/>
             <child link="${prefix}_thigh"/>
-            <dynamics damping="0.0" friction="0.001"/>
             <limit effort="${max_effort}" velocity="${max_velocity}" lower="-1e10" upper="1e10"/>
         </joint>
@@ -56,10 +55,4 @@
                    upper="${calf_upper_limit}"/>
         </joint>
-        <link name="${prefix}_foot"/>
-        <joint name="${prefix}_foot_fixed" type="fixed" dont_collapse="true">
-            <origin rpy="0 0 0" xyz="0 0 -0.27"/>
-            <parent link="${prefix}_calf"/>
-            <child link="${prefix}_foot"/>
-        </joint>
     </xacro:macro>
 </robot>
