Commit message: Add imu stl.

File: bipedal_wheel_description/urdf/imu.urdf.xacro (robot description, xacro)
@@ -18,5 +18,5 @@
                 <origin rpy="0 0 0" xyz="0 0 0"/>
                 <geometry>
-                    <mesh filename="package://rm_description/meshes/common/imu.stl" scale="1 1 1"/>
+                    <mesh filename="package://bipedal_wheel_description/meshes/imu.stl" scale="1 1 1"/>
                 </geometry>
             </visual>
