Commit message: Add LQR controller and modify some path.

File: bipedal_wheel_description/urdf/bipedal.urdf.xacro (robot description, xacro)
@@ -3,5 +3,5 @@
     <xacro:arg name="use_simulation" default="true"/>
     <xacro:arg name="add_wheel" default="false"/>
-    <xacro:include filename="$(find bipedal_description)/urdf/chassis.urdf.xacro"/>
+    <xacro:include filename="$(find bipedal_wheel_description)/urdf/chassis.urdf.xacro"/>
     <xacro:chassis use_simulation="$(arg use_simulation)" add_wheel="$(arg add_wheel)"/>
     <xacro:include filename="$(find rm_description)/urdf/common/imu.urdf.xacro"/>

File: bipedal_wheel_description/urdf/chassis.urdf.xacro (robot description, xacro)
@@ -11,6 +11,6 @@
     <xacro:property name="wheel_joint_effort" value="3.07"/>
     <xacro:property name="wheel_joint_velocity" value="73.6"/>
-    <xacro:include filename="$(find bipedal_description)/urdf/leg.urdf.xacro"/>
-    <xacro:include filename="$(find bipedal_description)/urdf/leg.transmission.xacro"/>
+    <xacro:include filename="$(find bipedal_wheel_description)/urdf/leg.urdf.xacro"/>
+    <xacro:include filename="$(find bipedal_wheel_description)/urdf/leg.transmission.xacro"/>
     <xacro:macro name="guide_wheel" params="prefix x_offset y_offset z_offset">
         <link name="${prefix}_guide_wheel">
@@ -49,5 +49,5 @@
                 <origin xyz="0 0 0" rpy="0 0 0"/>
                 <geometry>
-                    <mesh filename="package://bipedal_description/meshes/wheel.stl"/>
+                    <mesh filename="package://bipedal_wheel_description/meshes/wheel.stl"/>
                 </geometry>
             </visual>

File: bipedal_wheel_description/urdf/leg.urdf.xacro (robot description, xacro)
@@ -9,5 +9,5 @@
                 <origin xyz="0 0 0" rpy="0 0 0"/>
                 <geometry>
-                    <mesh filename="package://bipedal_description/meshes/first_leg.stl"/>
+                    <mesh filename="package://bipedal_wheel_description/meshes/first_leg.stl"/>
                 </geometry>
             </visual>
@@ -31,5 +31,5 @@
                 <origin xyz="0 0 0" rpy="0 0 0"/>
                 <geometry>
-                    <mesh filename="package://bipedal_description/meshes/second_leg.stl"/>
+                    <mesh filename="package://bipedal_wheel_description/meshes/second_leg.stl"/>
                 </geometry>
             </visual>
@@ -37,5 +37,5 @@
                 <origin xyz="0 0 0.0" rpy="0 0 0"/>
                 <geometry>
-                    <mesh filename="package://bipedal_description/meshes/second_leg.stl"/>
+                    <mesh filename="package://bipedal_wheel_description/meshes/second_leg.stl"/>
                 </geometry>
             </collision>

Commit message: Add radar.

File: bipedal_wheel_description/urdf/bipedal.urdf.xacro (robot description, xacro)
@@ -3,4 +3,8 @@
     <xacro:arg name="use_simulation" default="true"/>
     <xacro:arg name="add_wheel" default="false"/>
+    <xacro:arg name="gpu" default="false"/>
+    <xacro:property name="gpu" value="$(arg gpu)"/>
+    <xacro:arg name="organize_cloud" default="false"/>
+    <xacro:property name="organize_cloud" value="$(arg organize_cloud)"/>
     <xacro:include filename="$(find bipedal_wheel_description)/urdf/chassis.urdf.xacro"/>
     <xacro:chassis use_simulation="$(arg use_simulation)" add_wheel="$(arg add_wheel)"/>
@@ -8,4 +12,9 @@
     <xacro:IMU connected_to="base_link" imu_name="base_imu" xyz="0 0 0"
                rpy="0 0 -${pi}"/>
+    <xacro:include filename="$(find velodyne_description)/urdf/VLP-16.urdf.xacro"/>
+    <xacro:VLP-16 parent="base_link" name="velodyne" topic="/velodyne_points" organize_cloud="${organize_cloud}" hz="10"
+                  samples="440" gpu="${gpu}">
+        <origin xyz="0 0 0.08" rpy="0 0 0"/>
+    </xacro:VLP-16>
     <xacro:if value="$(arg use_simulation)">
         <gazebo>

Commit message: Modify params.

File: bipedal_wheel_description/urdf/bipedal.urdf.xacro (robot description, xacro)
@@ -15,5 +15,5 @@
     <xacro:VLP-16 parent="base_link" name="velodyne" topic="/velodyne_points" organize_cloud="${organize_cloud}" hz="10"
                   samples="1875" min_range="0.1" gpu="${gpu}">
-        <origin xyz="0 0 0.08" rpy="0 0 0"/>
+        <origin xyz="0 0 0.11" rpy="0 0 0"/>
     </xacro:VLP-16>
     <xacro:if value="$(arg use_simulation)">
@@ -24,4 +24,16 @@
             </plugin>
         </gazebo>
+        <gazebo>
+            <plugin name="p3d_base_controller" filename="libgazebo_ros_p3d.so">
+                <alwaysOn>true</alwaysOn>
+                <updateRate>500.0</updateRate>
+                <bodyName>base_link</bodyName>
+                <topicName>ground_truth/state</topicName>
+                <gaussianNoise>0.0</gaussianNoise>
+                <frameName>world</frameName>
+                <xyzOffsets>0 0 0</xyzOffsets>
+                <rpyOffsets>0 0 0</rpyOffsets>
+            </plugin>
+        </gazebo>
     </xacro:if>
 </robot>

File: bipedal_wheel_description/urdf/chassis.urdf.xacro (robot description, xacro)
@@ -9,6 +9,6 @@
     <xacro:property name="wheel_radius" value="0.09"/>
     <xacro:property name="wheel_z_offset" value="-0.270"/>
-    <xacro:property name="wheel_joint_effort" value="3.07"/>
-    <xacro:property name="wheel_joint_velocity" value="73.6"/>
+    <xacro:property name="wheel_joint_effort" value="5"/>
+    <xacro:property name="wheel_joint_velocity" value="50"/>
     <xacro:include filename="$(find bipedal_wheel_description)/urdf/leg.urdf.xacro"/>
     <xacro:include filename="$(find bipedal_wheel_description)/urdf/leg.transmission.xacro"/>
@@ -116,13 +116,13 @@
             <xacro:wheel connected_to="left_calf" prefix="left" wheel_x_offset="0"
                          wheel_y_offset="${wheel_base/2-leg_y_offset}"
-                         wheel_z_offset="${wheel_z_offset}" mechanical_reduction="-13"/>
+                         wheel_z_offset="${wheel_z_offset}" mechanical_reduction="-19.2032"/>
             <xacro:wheel connected_to="right_calf" prefix="right" wheel_x_offset="0"
                          wheel_y_offset="${-(wheel_base/2-leg_y_offset)}"
-                         wheel_z_offset="${wheel_z_offset}" mechanical_reduction="13"/>
+                         wheel_z_offset="${wheel_z_offset}" mechanical_reduction="19.2032"/>
         </xacro:if>
-        <xacro:guide_wheel prefix="left_front" x_offset="0.24" y_offset="0.1" z_offset="-0.08"/>
-        <xacro:guide_wheel prefix="right_front" x_offset="0.24" y_offset="-0.1" z_offset="-0.08"/>
-        <xacro:guide_wheel prefix="left_back" x_offset="-0.24" y_offset="0.1" z_offset="-0.08"/>
-        <xacro:guide_wheel prefix="right_back" x_offset="-0.24" y_offset="-0.1" z_offset="-0.08"/>
+<!--        <xacro:guide_wheel prefix="left_front" x_offset="0.24" y_offset="0.1" z_offset="-0.08"/>-->
+<!--        <xacro:guide_wheel prefix="right_front" x_offset="0.24" y_offset="-0.1" z_offset="-0.08"/>-->
+<!--        <xacro:guide_wheel prefix="left_back" x_offset="-0.24" y_offset="0.1" z_offset="-0.08"/>-->
+<!--        <xacro:guide_wheel prefix="right_back" x_offset="-0.24" y_offset="-0.1" z_offset="-0.08"/>-->
     </xacro:macro>
 </robot>

Commit message: Update urdf.

File: bipedal_wheel_description/urdf/bipedal.urdf.xacro (robot description, xacro)
@@ -11,10 +11,13 @@
     <xacro:include filename="$(find bipedal_wheel_description)/urdf/imu.urdf.xacro"/>
     <xacro:IMU connected_to="base_link" imu_name="base_imu" xyz="0 0 0"
-               rpy="0 0 -${pi}"/>
-    <xacro:include filename="$(find velodyne_description)/urdf/VLP-16.urdf.xacro"/>
-    <xacro:VLP-16 parent="base_link" name="velodyne" topic="/velodyne_points" organize_cloud="${organize_cloud}" hz="10"
-                  samples="1875" min_range="0.1" gpu="${gpu}">
-        <origin xyz="0 0 0.11" rpy="0 0 0"/>
-    </xacro:VLP-16>
+               rpy="0 0 0"/>
+    <!--    <xacro:include filename="$(find velodyne_description)/urdf/VLP-16.urdf.xacro"/>-->
+    <!--    <xacro:VLP-16 parent="base_link" name="velodyne" topic="/velodyne_points" organize_cloud="${organize_cloud}" hz="10"-->
+    <!--                  samples="1875" min_range="0.1" gpu="${gpu}">-->
+    <!--        <origin xyz="0 0 0.11" rpy="0 0 0"/>-->
+    <!--    </xacro:VLP-16>-->
+    <xacro:include filename="$(find bipedal_wheel_description)/urdf/livox_mid360.urdf.xacro"/>
+    <xacro:livox_mid360 connected_to="base_link" simulation="$(arg use_simulation)" lidar_name="livox_frame"
+                        xyz="0 0 0.12" rpy="0 0 0"/>
     <xacro:if value="$(arg use_simulation)">
         <gazebo>

File: bipedal_wheel_description/urdf/chassis.urdf.xacro (robot description, xacro)
@@ -2,16 +2,17 @@
 <robot xmlns:xacro="http://www.ros.org/wiki/xacro">
     <!-- https://upload.wikimedia.org/wikipedia/commons/5/52/Wheelbase_and_Track.png -->
-    <xacro:property name="wheel_base" value="0.4893"/>
     <xacro:property name="leg_x_offset" value="0.0"/>
-    <xacro:property name="leg_y_offset" value="0.208"/>
-    <xacro:property name="leg_z_offset" value="0."/>
+    <xacro:property name="leg_y_offset" value="0.178"/>
+    <xacro:property name="leg_z_offset" value="0.038"/>
     <xacro:property name="leg_pitch_offset" value="${pi/2}"/>
-    <xacro:property name="wheel_radius" value="0.09"/>
-    <xacro:property name="wheel_z_offset" value="-0.270"/>
+    <xacro:property name="second_leg_y_offset" value="0.018"/>
+    <xacro:property name="wheel_radius" value="0.055"/>
+    <xacro:property name="wheel_y_offset" value="0.05"/>
+    <xacro:property name="wheel_z_offset" value="-0.26"/>
     <xacro:property name="wheel_joint_effort" value="5"/>
     <xacro:property name="wheel_joint_velocity" value="50"/>
     <xacro:include filename="$(find bipedal_wheel_description)/urdf/leg.urdf.xacro"/>
     <xacro:include filename="$(find bipedal_wheel_description)/urdf/leg.transmission.xacro"/>
-    <xacro:macro name="guide_wheel" params="prefix x_offset y_offset z_offset">
+    <xacro:macro name="guide_wheel" params="connected_to prefix x_offset y_offset z_offset">
         <link name="${prefix}_guide_wheel">
             <visual>
@@ -30,14 +31,13 @@
                 <mass value="0.05"/>
                 <origin xyz="0 0 0"/>
-                <inertia ixx="1.752e-3" ixy="-2.766e-6" ixz="-1.599e-6" iyy="3.357e-3"
-                         iyz="2.581e-6" izz="1.752e-3"/>
+                <inertia ixx="5.417e-6" ixy="0.0" ixz="0.0" iyy="1.0e-5" iyz="0.0" izz="5.417e-6"/>
             </inertial>
         </link>
         <joint name="${prefix}_guide_wheel_joint" type="revolute">
-            <parent link="base_link"/>
+            <parent link="${connected_to}"/>
             <child link="${prefix}_guide_wheel"/>
             <origin xyz="${x_offset} ${y_offset} ${z_offset}" rpy="0 0 0"/>
             <limit effort="0." velocity="99" lower="-1e16" upper="1e16"/>
-            <dynamics damping="0.05" friction="0.05"/>
+            <dynamics damping="0.0" friction="0.05"/>
             <axis xyz="0 1 0"/>
         </joint>
@@ -70,4 +70,5 @@
             <parent link="${connected_to}"/>
             <child link="${prefix}_wheel"/>
+            <dynamics damping="0.0" friction="0.08"/>
             <limit effort="${wheel_joint_effort}" velocity="${wheel_joint_velocity}" lower="-1e16" upper="1e16"/>
         </joint>
@@ -86,43 +87,52 @@
             <inertial>
                 <mass value="11.70"/>
-                <origin xyz="0.0033 0.006725 -0.013651"/>
-                <inertia ixx="2.56e-1" ixy="1.044e-3" ixz="1.56e-2" iyy="1.748e-1"
-                         iyz="-7.548e-4" izz="3.787e-1"/>
+                <origin xyz="0 0 0"/>
+                <inertia ixx="0.085" ixy="0.0" ixz="0.0" iyy="0.085" iyz="0.0" izz="0.132"/>
             </inertial>
             <visual>
                 <origin xyz="0 0 0" rpy="0 0 0"/>
                 <geometry>
-                    <cylinder length="0.15" radius="0.18"/>
+                    <cylinder length="0.14" radius="0.15"/>
                 </geometry>
             </visual>
             <collision>
-                <origin xyz="0 0.008 0" rpy="0 0 0"/>
+                <origin xyz="0 0.0 0" rpy="0 0 0"/>
                 <geometry>
-                    <box size="0.482 0.332 0.183"/>
+                    <cylinder length="0.14" radius="0.15"/>
                 </geometry>
             </collision>
         </link>
         <xacro:leg prefix="left" connected_to="base_link" pitch_offset="${leg_pitch_offset}"
-                   leg_x_offset="${-leg_x_offset}"
+                   leg_x_offset="${leg_x_offset}"
                    leg_y_offset="${leg_y_offset}"
-                   leg_z_offset="${leg_z_offset}"/>
+                   leg_z_offset="${leg_z_offset}"
+                   second_leg_y_offset="${second_leg_y_offset}"/>
         <xacro:leg prefix="right" connected_to="base_link" pitch_offset="${leg_pitch_offset}"
-                   leg_x_offset="${-leg_x_offset}"
-                   leg_y_offset="${-leg_y_offset}"
-                   leg_z_offset="${leg_z_offset}"/>
+                   leg_x_offset="${leg_x_offset}"
+                   leg_y_offset="-${leg_y_offset}"
+                   leg_z_offset="${leg_z_offset}"
+                   second_leg_y_offset="-${second_leg_y_offset}"/>
         <xacro:leg_transmission prefix="left" mechanical_reduction="-1"/>
         <xacro:leg_transmission prefix="right" mechanical_reduction="1"/>
         <xacro:if value="${add_wheel}">
             <xacro:wheel connected_to="left_calf" prefix="left" wheel_x_offset="0"
-                         wheel_y_offset="${wheel_base/2-leg_y_offset}"
+                         wheel_y_offset="${wheel_y_offset}"
                          wheel_z_offset="${wheel_z_offset}" mechanical_reduction="-19.2032"/>
             <xacro:wheel connected_to="right_calf" prefix="right" wheel_x_offset="0"
-                         wheel_y_offset="${-(wheel_base/2-leg_y_offset)}"
+                         wheel_y_offset="${-wheel_y_offset}"
                          wheel_z_offset="${wheel_z_offset}" mechanical_reduction="19.2032"/>
         </xacro:if>
-        <xacro:guide_wheel prefix="left_front" x_offset="0.24" y_offset="0.1" z_offset="-0.08"/>
-        <xacro:guide_wheel prefix="right_front" x_offset="0.24" y_offset="-0.1" z_offset="-0.08"/>
-        <xacro:guide_wheel prefix="left_back" x_offset="-0.24" y_offset="0.1" z_offset="-0.08"/>
-        <xacro:guide_wheel prefix="right_back" x_offset="-0.24" y_offset="-0.1" z_offset="-0.08"/>
+        <xacro:guide_wheel connected_to="base_link" prefix="left_front" x_offset="0.16" y_offset="0.08"
+                           z_offset="-0.07"/>
+        <xacro:guide_wheel connected_to="base_link" prefix="right_front" x_offset="0.16" y_offset="-0.08"
+                           z_offset="-0.07"/>
+        <xacro:guide_wheel connected_to="base_link" prefix="left_back" x_offset="-0.16" y_offset="0.08"
+                           z_offset="-0.07"/>
+        <xacro:guide_wheel connected_to="base_link" prefix="right_back" x_offset="-0.16" y_offset="-0.08"
+                           z_offset="-0.07"/>
+        <!--        <xacro:guide_wheel connected_to="left_calf" prefix="left_calf" x_offset="-0.01" y_offset="0.02"-->
+        <!--                           z_offset="0.07"/>-->
+        <!--        <xacro:guide_wheel connected_to="right_calf" prefix="right_calf" x_offset="-0.01" y_offset="-0.02"-->
+        <!--                           z_offset="0.07"/>-->
     </xacro:macro>
 </robot>

File: bipedal_wheel_description/urdf/leg.urdf.xacro (robot description, xacro)
@@ -3,18 +3,24 @@
     <xacro:property name="max_velocity" value="10.46"/>
     <xacro:property name="calf_upper_limit" value="0."/>
-    <xacro:property name="calf_lower_limit" value="-2."/>
-    <xacro:macro name="leg" params="prefix connected_to pitch_offset leg_x_offset leg_y_offset leg_z_offset">
+    <xacro:property name="calf_lower_limit" value="-1.85"/>
+    <xacro:macro name="leg"
+                 params="prefix connected_to pitch_offset leg_x_offset leg_y_offset leg_z_offset second_leg_y_offset">
         <link name="${prefix}_thigh">
             <visual>
-                <origin xyz="0 0 0" rpy="0 0 0"/>
+                <origin xyz="0 -0.005 0" rpy="0 0 0"/>
                 <geometry>
                     <mesh filename="package://bipedal_wheel_description/meshes/first_leg.stl"/>
                 </geometry>
             </visual>
+            <collision>
+                <origin xyz="0 0 -0.1"/>
+                <geometry>
+                    <box size="0.06 0.013 0.2"/>
+                </geometry>
+            </collision>
             <inertial>
-                <mass value="0.116"/>
-                <origin xyz="0.000354 0.006 -0.067161"/>
-                <inertia ixx="3.922e-4" ixy="-9.1e-12" ixz="4.457e-6" iyy="4.316e-4" iyz="1.581e-9"
-                         izz="4.2181e-5"/>
+                <mass value="0.164"/>
+                <origin xyz="0 0 -0.109"/>
+                <inertia ixx="6.51e-4" ixy="0.0" ixz="0.0" iyy="6.56e-4" iyz="0.0" izz="5.47e-5"/>
             </inertial>
         </link>
@@ -25,9 +31,8 @@
             <child link="${prefix}_thigh"/>
             <limit effort="${max_effort}" velocity="${max_velocity}" lower="-1e10" upper="1e10"/>
-            <safety_controller k_position="100" k_velocity="1" soft_lower_limit="-1e10" soft_upper_limit="1e10"/>
         </joint>
         <link name="${prefix}_calf">
             <visual>
-                <origin xyz="0 0 0" rpy="0 0 0"/>
+                <origin xyz="0 -0.005 0" rpy="0 0 0"/>
                 <geometry>
                     <mesh filename="package://bipedal_wheel_description/meshes/second_leg.stl"/>
@@ -35,24 +40,25 @@
             </visual>
             <collision>
-                <origin xyz="0 0 0.0" rpy="0 0 0"/>
+                <origin xyz="0 0 -0.13" rpy="0 0 0"/>
                 <geometry>
-                    <mesh filename="package://bipedal_wheel_description/meshes/second_leg.stl"/>
+                    <box size="0.06 0.013 0.25"/>
                 </geometry>
             </collision>
             <inertial>
-                <mass value="0.193603"/>
-                <origin xyz="0.000074 0.006 -0.123983"/>
-                <inertia ixx="1.639e-3" ixy="-1.067e-16" ixz="6.533e-7" iyy="1.709e-3" iyz="0.0"
-                         izz="7.4906e-5"/>
+                <mass value="0.190142"/>
+                <origin xyz="0.0000 0.00 -0.12"/>
+                <inertia ixx="1.976e-3" ixy="-5.117e-9" ixz="3.239e-6" iyy="2.024e-3" iyz="2.338e-6"
+                         izz="5.2689e-5"/>
             </inertial>
         </link>
         <joint name="${prefix}_knee_joint" type="revolute">
             <axis xyz="0 1 0"/>
-            <origin xyz="0 0 -0.15" rpy="0 -${pi/4} 0"/>
+            <origin xyz="0 ${second_leg_y_offset} -0.218" rpy="0 -${pi/4} 0"/>
             <parent link="${prefix}_thigh"/>
             <child link="${prefix}_calf"/>
-            <dynamics damping="0.0" friction="0.001"/>
             <limit effort="${max_effort}" velocity="${max_velocity}" lower="${calf_lower_limit}"
                    upper="${calf_upper_limit}"/>
+            <!--            <safety_controller k_position="10" k_velocity="0.1" soft_lower_limit="${calf_lower_limit}"-->
+            <!--                               soft_upper_limit="1e10"/>-->
         </joint>
     </xacro:macro>

Commit message: Use velodyne.

File: bipedal_wheel_description/urdf/bipedal.urdf.xacro (robot description, xacro)
@@ -12,12 +12,12 @@
     <xacro:IMU connected_to="base_link" imu_name="base_imu" xyz="0 0 0"
                rpy="0 0 0"/>
-    <!--    <xacro:include filename="$(find velodyne_description)/urdf/VLP-16.urdf.xacro"/>-->
-    <!--    <xacro:VLP-16 parent="base_link" name="velodyne" topic="/velodyne_points" organize_cloud="${organize_cloud}" hz="10"-->
-    <!--                  samples="1875" min_range="0.1" gpu="${gpu}">-->
-    <!--        <origin xyz="0 0 0.11" rpy="0 0 0"/>-->
-    <!--    </xacro:VLP-16>-->
-    <xacro:include filename="$(find bipedal_wheel_description)/urdf/livox_mid360.urdf.xacro"/>
-    <xacro:livox_mid360 connected_to="base_link" simulation="$(arg use_simulation)" lidar_name="livox_frame"
-                        xyz="0 0 0.12" rpy="0 0 0"/>
+    <xacro:include filename="$(find velodyne_description)/urdf/VLP-16.urdf.xacro"/>
+    <xacro:VLP-16 parent="base_link" name="velodyne" topic="/velodyne_points" organize_cloud="${organize_cloud}" hz="10"
+                  samples="1875" min_range="0.1" gpu="${gpu}">
+        <origin xyz="0 0 0.11" rpy="0 0 0"/>
+    </xacro:VLP-16>
+    <!--    <xacro:include filename="$(find bipedal_wheel_description)/urdf/livox_mid360.urdf.xacro"/>-->
+    <!--    <xacro:livox_mid360 connected_to="base_link" simulation="$(arg use_simulation)" lidar_name="livox_frame"-->
+    <!--                        xyz="0 0 0.12" rpy="0 0 0"/>-->
     <xacro:if value="$(arg use_simulation)">
         <gazebo>
